File: Xen40/Xen40.sch (KiCad schematic (older format))
At the start: 23 parts

Commit message: new files
Parts:
- added D47: G-LED, LED_SMD:LED_0805_2012Metric_Pad1.15x1.40mm_HandSolder, symbol Device:LED
- added F1: 500mA, Fuse:Fuse_1206_3216Metric_Pad1.42x1.75mm_HandSolder, symbol Device:Polyfuse_Small
- added H1, H2: MountingHole, random-keyboard-parts:MOUNTINGHOLE_2.5_PLATED, symbol Mechanical:MountingHole
- added J1: USB SMD Header, random-keyboard-parts:S4B-ZR, symbol Connector_Generic:Conn_01x04
- added J2: BLE TH Header, random-keyboard-parts:1X09_ROUND_70, symbol Connector_Generic:Conn_01x09
- added J3: OLED Header, random-keyboard-parts:OLED_4Pin, symbol Connector_Generic:Conn_01x04
- added J4: BATT Header, random-keyboard-parts:S2B-PH-K-S, symbol Connector_Generic:Conn_01x02
- added R8: 470, Resistor_SMD:R_0805_2012Metric_Pad1.15x1.40mm_HandSolder, symbol Device:R_Small_US
- C1, C10, C2, C3, C4, C5, C6, C7, C8, C9: renamed from C?; footprint (none) -> Capacitor_SMD:C_0805_2012Metric
- D1: renamed from D?; value MBR120 (NEEDS FOOTPRINT & SYMBOL) -> MBR120; footprint (none) -> Diode_SMD:D_SOD-123
- D2: renamed from D?; value LED -> O-LED; footprint (none) -> LED_SMD:LED_0805_2012Metric_Pad1.15x1.40mm_HandSolder
- R1, R2, R3, R4, R5: renamed from R?; footprint (none) -> Resistor_SMD:R_0805_2012Metric_Pad1.15x1.40mm_HandSolder
- R6: renamed from R?; value 1k -> 470; footprint (none) -> Resistor_SMD:R_0805_2012Metric_Pad1.15x1.40mm_HandSolder
- SW1: renamed from SW?; footprint (none) -> random-keyboard-parts:SKQG-1155865
- Y1: renamed from Y?; footprint (none) -> Crystal:Crystal_SMD_3225-4Pin_3.2x2.5mm_HandSoldering
- gave numbers to parts that had none: 3
Connections:
- net labels added: +5V, BLE_DFU, Col1, Col10, Col11, Col12, Col2, Col3, Col4, Col5, Col6, Col7, Col8, Col9, Row1, Row2, Row3, Row4
- wire segments 101 -> 155
- no-connect marks 2 -> 3
Other:
- note removed: "Connect BLE_DFU to 0 ohm res\n"
- note removed: "NEED OLED_RST???\n"
- moved on the sheet: C1, C10, C2, C3, C4, C5, C6, C7, C8, C9, D1, D2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

Commit message: Finished Initial Routing for V1
Parts:
- added SW2: SW_SPDT, random-keyboard-parts:Batt_SW, symbol Switch:SW_SPDT
Connections:
- net labels added: +VSW
- wire segments 155 -> 175
- no-connect marks 3 -> 4
Changed lines of the file:
@@
 	0    1    1    0
-$EndComp
-$Comp
-L power:+BATT #PWR0106
-U 1 1 5E7B9DBE
-P 9350 4000
-F 0 "#PWR0106" H 9350 3850 50  0001 C CNN
-F 1 "+BATT" H 9365 4173 50  0000 C CNN
-F 2 "" H 9350 4000 50  0001 C CNN
-F 3 "" H 9350 4000 50  0001 C CNN
-	1    9350 4000
-	1    0    0    -1
 $EndComp
 Connection ~ 8850 4800
@@
 Wire Wire Line
 	8000 5200 8000 5300
-$Comp
-L power:+BATT #PWR0110
-U 1 1 5E775143
-P 8000 5200
-F 0 "#PWR0110" H 8000 5050 50  0001 C CNN
-F 1 "+BATT" H 8015 5373 50  0000 C CNN
-F 2 "" H 8000 5200 50  0001 C CNN
-F 3 "" H 8000 5200 50  0001 C CNN
-	1    8000 5200
-	1    0    0    -1
-$EndComp
 $Comp
 L Device:D_Schottky_Small D1
@@
 $EndSheet
 Wire Wire Line
-	9800 1100 9400 1100
-Wire Wire Line
-	9400 1200 9800 1200
-Wire Wire Line
-	9800 1300 9400 1300
-Wire Wire Line
-	9800 1400 9400 1400
-Wire Wire Line
 	9400 1600 9800 1600
 Wire Wire Line
@@
 Wire Wire Line
 	9400 2500 9800 2500
-Text GLabel 9400 1100 0    50   Input ~ 0
-Row1
-Text GLabel 9400 1200 0    50   Input ~ 0
-Row2
-Text GLabel 9400 1300 0    50   Input ~ 0
-Row3
-Text GLabel 9400 1400 0    50   Input ~ 0
-Row4
-Text GLabel 9400 1600 0    50   Input ~ 0
-Col1
-Text GLabel 9400 1700 0    50   Input ~ 0
-Col2
-Text GLabel 9400 1800 0    50   Input ~ 0
-Col3
-Text GLabel 9400 1900 0    50   Input ~ 0
-Col4
-Text GLabel 9400 2000 0    50   Input ~ 0
-Col5
-Text GLabel 9400 2100 0    50   Input ~ 0
-Col6
-Text GLabel 9400 2200 0    50   Input ~ 0
-Col7
-Text GLabel 9400 2300 0    50   Input ~ 0
-Col8
-Text GLabel 9400 2400 0    50   Input ~ 0
-Col9
-Text GLabel 9400 2500 0    50   Input ~ 0
-Col10
 $Comp
 L Connector_Generic:Conn_01x04 J1
@@
 Wire Wire Line
 	2300 7200 1300 7200
-Text GLabel 9400 2600 0    50   Input ~ 0
-Col11
 Wire Wire Line
 	9400 2600 9800 2600
-Text GLabel 9400 2700 0    50   Input ~ 0
-Col12
 Wire Wire Line
 	9400 2700 9800 2700
@@
 	4050 7000 3150 7000
 NoConn ~ 4050 7000
+$Comp
+L Switch:SW_SPDT SW2
+U 1 1 5EBDDC71
+P 4500 5850
+F 0 "SW2" H 4500 6135 50  0000 C CNN
+F 1 "SW_SPDT" H 4500 6044 50  0000 C CNN
+F 2 "random-keyboard-parts:Batt_SW" H 4500 5850 50  0001 C CNN
+F 3 "~" H 4500 5850 50  0001 C CNN
+	1    4500 5850
+	1    0    0    -1
+$EndComp
+$Comp
+L power:+BATT #PWR0106
+U 1 1 5EBE7CC9
+P 4050 5800
+F 0 "#PWR0106" H 4050 5650 50  0001 C CNN
+F 1 "+BATT" H 4065 5973 50  0000 C CNN
+F 2 "" H 4050 5800 50  0001 C CNN
+F 3 "" H 4050 5800 50  0001 C CNN
+	1    4050 5800
+	1    0    0    -1
+$EndComp
+Wire Wire Line
+	4050 5800 4050 5850
+Wire Wire Line
+	4050 5850 4300 5850
+$Comp
+L power:+VSW #PWR0110
+U 1 1 5EBF16B7
+P 4950 5700
+F 0 "#PWR0110" H 4950 5550 50  0001 C CNN
+F 1 "+VSW" H 4965 5873 50  0000 C CNN
+F 2 "" H 4950 5700 50  0001 C CNN
+F 3 "" H 4950 5700 50  0001 C CNN
+	1    4950 5700
+	1    0    0    -1
+$EndComp
+Wire Wire Line
+	4950 5700 4950 5750
+Wire Wire Line
+	4950 5750 4700 5750
+NoConn ~ 4700 5950
+$Comp
+L power:+VSW #PWR0130
+U 1 1 5EC01863
+P 9350 4000
+F 0 "#PWR0130" H 9350 3850 50  0001 C CNN
+F 1 "+VSW" H 9365 4173 50  0000 C CNN
+F 2 "" H 9350 4000 50  0001 C CNN
+F 3 "" H 9350 4000 50  0001 C CNN
+	1    9350 4000
+	1    0    0    -1
+$EndComp
+$Comp
+L power:+VSW #PWR0131
+U 1 1 5EC02FC3
+P 8000 5200
+F 0 "#PWR0131" H 8000 5050 50  0001 C CNN
+F 1 "+VSW" H 8015 5373 50  0000 C CNN
+F 2 "" H 8000 5200 50  0001 C CNN
+F 3 "" H 8000 5200 50  0001 C CNN
+	1    8000 5200
+	1    0    0    -1
+$EndComp
+Text GLabel 9400 1400 0    50   Input ~ 0
+Row4
+Text GLabel 9400 1300 0    50   Input ~ 0
+Row3
+Text GLabel 9400 1200 0    50   Input ~ 0
+Row2
+Text GLabel 9400 1100 0    50   Input ~ 0
+Row1
+Wire Wire Line
+	9800 1400 9400 1400
+Wire Wire Line
+	9800 1300 9400 1300
+Wire Wire Line
+	9400 1200 9800 1200
+Wire Wire Line
+	9800 1100 9400 1100
+Text GLabel 4800 4050 2    50   Output ~ 0
+Row1
+Text GLabel 4800 3950 2    50   Output ~ 0
+Row2
+Text GLabel 4800 3850 2    50   Output ~ 0
+Row3
+Text GLabel 4800 1450 2    50   Output ~ 0
+Row4
+Text GLabel 9400 2700 0    50   Input ~ 0
+Col12
+Text GLabel 9400 2600 0    50   Input ~ 0
+Col11
+Text GLabel 9400 2500 0    50   Input ~ 0
+Col10
+Text GLabel 9400 2400 0    50   Input ~ 0
+Col9
+Text GLabel 9400 2300 0    50   Input ~ 0
+Col8
+Text GLabel 9400 2200 0    50   Input ~ 0
+Col7
+Text GLabel 9400 2100 0    50   Input ~ 0
+Col6
+Text GLabel 9400 2000 0    50   Input ~ 0
+Col5
+Text GLabel 9400 1900 0    50   Input ~ 0
+Col4
+Text GLabel 9400 1800 0    50   Input ~ 0
+Col3
+Text GLabel 9400 1700 0    50   Input ~ 0
+Col2
+Text GLabel 9400 1600 0    50   Input ~ 0
+Col1
+Text GLabel 4800 2850 2    50   Output ~ 0
+Col1
+Text GLabel 4800 2950 2    50   Output ~ 0
+Col2
+Text GLabel 4800 3150 2    50   Output ~ 0
+Col3
+Text GLabel 4800 3250 2    50   Output ~ 0
+Col4
+Text GLabel 4800 3350 2    50   Output ~ 0
+Col5
+Text GLabel 4800 1950 2    50   Output ~ 0
+Col6
+Text GLabel 4800 2050 2    50   Output ~ 0
+Col7
+Text GLabel 4800 2350 2    50   Output ~ 0
+Col8
+Text GLabel 4800 2450 2    50   Output ~ 0
+Col9
+Text GLabel 4800 4350 2    50   Output ~ 0
+Col10
+Text GLabel 4800 4250 2    50   Output ~ 0
+Col11
+Text GLabel 4800 4150 2    50   Output ~ 0
+Col12
+Wire Wire Line
+	4800 4050 4050 4050
+Wire Wire Line
+	4050 3950 4800 3950
+Wire Wire Line
+	4800 3850 4050 3850
+Wire Wire Line
+	4800 4150 4050 4150
+Wire Wire Line
+	4050 4250 4800 4250
+Wire Wire Line
+	4800 4350 4050 4350
+Wire Wire Line
+	4800 1950 4050 1950
+Wire Wire Line
+	4800 2050 4050 2050
+Wire Wire Line
+	4050 2350 4800 2350
+Wire Wire Line
+	4800 2450 4050 2450
+Wire Wire Line
+	4800 2850 4050 2850
+Wire Wire Line
+	4050 2950 4800 2950
+Wire Wire Line
+	4800 3150 4050 3150
+Wire Wire Line
+	4050 3250 4800 3250
+Wire Wire Line
+	4800 3350 4050 3350
+Wire Wire Line
+	4800 1450 4050 1450
 $EndSCHEMATC
